Commit message: Fixed Arm Physics
Ahora puede girar con un rango mas amplio el brazo

File: simulation/models/jag.urdf (robot description, URDF)
Before this commit: robot jaguar, 18 links, 17 joints
Joints:
- joint arm_2_hinge: limit lower=-2.9 upper=2.9 effort=10000 velocity=0.05 -> lower=-15.6 upper=15.6 effort=10000 velocity=0.05

Commit message: Fixed Collision Arm1 & Arm2
Ahora las fisicas del arm1  y arm2 están disponibles

File: simulation/models/jag.urdf (robot description, URDF)
Before this commit: robot jaguar, 18 links, 17 joints
Links:
- link arm_1: geometry collision cylinder length=0.34 radius=0.025; visual mesh filename=package://simulation/models/meshes/jaguar/arm1.dae scale=0.021 0.021 0.021
- link arm_2: geometry collision cylinder length=0.15 radius=0.025; visual mesh filename=package://simulation/models/meshes/jaguar/arm2.dae scale=0.021 0.021 0.021
- link arm_3: geometry collision cylinder length=0.15 radius=0.025; visual mesh filename=package://simulation/models/meshes/jaguar/arm3.dae scale=0.021 0.021 0.021

Commit message: Changes in Joy & Camera
Se agrego el control del brazo por medio del Joystick y la posicion de la camara (base y brazo).

File: simulation/models/jag.urdf (robot description, URDF)
Before this commit: robot jaguar, 18 links, 17 joints
Links:
- added link camera_depth_frame_2
- added link camera_depth_optical_frame_2
- added link camera_link_2; collision box size=0 0 0; visual box size=0 0 0
- added link camera_rgb_frame_2
- added link camera_rgb_optical_frame_2
- link arm_1: geometry visual mesh filename=package://simulation/models/meshes/jaguar/arm1.dae scale=0.021 0.021 0.021
- link arm_2: geometry visual mesh filename=package://simulation/models/meshes/jaguar/arm2.dae scale=0.021 0.021 0.021
- link arm_3: geometry visual mesh filename=package://simulation/models/meshes/jaguar/arm3.dae scale=0.021 0.021 0.021
Joints:
- added joint camera_depth_joint_2: type fixed, parent camera_link_2, child camera_depth_frame_2, origin xyz=0.0 -0.02 0.0 rpy=0 0 0
- added joint camera_depth_optical_joint_2: type fixed, parent camera_depth_frame_2, child camera_depth_optical_frame_2, origin xyz=0 0 0 rpy=-1.57 0.0 -1.57
- added joint camera_joint_2: type fixed, parent arm_2, child camera_link_2, origin xyz=0.195 0.1 0.295 rpy=0 -1.60 0.0
- added joint camera_rgb_joint_2: type fixed, parent camera_link_2, child camera_rgb_frame_2, origin xyz=0.0 -0.0125 0.0 rpy=0 0 0
- added joint camera_rgb_optical_joint_2: type fixed, parent camera_rgb_frame_2, child camera_rgb_optical_frame_2, origin xyz=0 0 0 rpy=-1.57 0.0 -1.57
- joint camera_joint: origin xyz=0.195 0.1 0.295 rpy=0 0.46 0.0 -> xyz=0.195 0.1 0.295 rpy=0 0.00 0.0

Commit message: 3rd  Camera Added
Se añadio la tercer camara con vista hacia los flippers

File: simulation/models/jag.urdf (robot description, URDF)
Before this commit: robot jaguar, 23 links, 22 joints
Links:
- added link camera_depth_frame_3
- added link camera_depth_optical_frame_3
- added link camera_link_3; collision box size=0 0 0; visual box size=0 0 0
- added link camera_rgb_frame_3
- added link camera_rgb_optical_frame_3
Joints:
- added joint camera_depth_joint_3: type fixed, parent camera_link_3, child camera_depth_frame_3, origin xyz=0.0 0.00 0.0 rpy=0 0 0
- added joint camera_depth_optical_joint_3: type fixed, parent camera_depth_frame_3, child camera_depth_optical_frame_3, origin xyz=0 0 0 rpy=-0.1 0.0 -0.1
- added joint camera_joint_3: type fixed, parent base_link, child camera_link_3, origin xyz=-0.05 0.0 0.55 rpy=0.0 1.5 0.0
- added joint camera_rgb_joint_3: type fixed, parent camera_link_3, child camera_rgb_frame_3, origin xyz=0.0 -0.0125 0.0 rpy=0 0 0
- added joint camera_rgb_optical_joint_3: type fixed, parent camera_rgb_frame_3, child camera_rgb_optical_frame_3, origin xyz=0 0 0 rpy=-1.57 0.0 -1.57
